File: H19R00/H19R00.sch (EAGLE design)
At the start: 17 parts, among them U1 STM32G0B1CEU6N, X1 8MHZ

Commit message: -Adding the Original Files that has been designed by the Designer
Parts:
- added BOOT0, GND, SWDCLK, SWDIO: PAD4, HEXABITZ_CONNECTION_PARTS:PAD4
- added C10, C8, C9: 470nF, HEXABITZ_RCLS:C-0603
- added C11, C15, C16: 150nF, HEXABITZ_RCLS:C-0805
- added C12, C13: 10uF, HEXABITZ_RCLS:C-0805
- added C14, C17, C18: 33pF, HEXABITZ_RCLS:C-0603
- added C19, C26, C27: 1nF, HEXABITZ_RCLS:C-0603
- added C20: 47uF, HEXABITZ_RCLS:C-0805
- added C21, C22, C23: 100nF, HEXABITZ_RCLS:C-0603
- added C24, C25: 1uF, HEXABITZ_RCLS:C-0603
- added C28, C29, C46: 220pF, HEXABITZ_RCLS:C-0603
- added C30, C31: 47uF, HEXABITZ_RCLS:A780EN476M1HLAS050
- added C32, C33: 10nF, HEXABITZ_RCLS:C-0603
- added C45: 2.2nF, HEXABITZ_RCLS:C-0603
- added D10: RED, HEXABITZ_USER_INTERFACE_PARTS:VLMS1300-GS08
- added D2, D3, D4, D5, D6, D7: BAT30KFILM, HEXABITZ_RCLS:BAT30KFILM
- added D8: MMSD4448ONSEMI_MMSD4448_0_0, HEXABITZ_RCLS:MMSD4448ONSEMI_MMSD4448_0_0
- added FB2: 22uH, HEXABITZ_RCLS:FB-0805
- added J1: 691213710003, HEXABITZ_CONNECTION_PARTS:691213710003
- added J2: 691213710002, HEXABITZ_CONNECTION_PARTS:691213710002
- added J3: 20021121-00008T4LFU, HEXABITZ_CONNECTION_PARTS:20021121-00008T4LFU
- added J4: 20021121-00006C1LF, HEXABITZ_CONNECTION_PARTS:20021121-00006C1LF
- added Q1, Q2, Q3: (no value), HEXABITZ_ICs:PJQ5866A_R2_00001
- added R10, R14, R17: 0.100R, HEXABITZ_RCLS:R_1206R1206
- added R11, R13, R15, R16, R4, R5: 100, HEXABITZ_RCLS:R-0603
- added R12: 750K, HEXABITZ_RCLS:R-0603
- added R18, R20, R40, R43, R45, R8: 2.4K, HEXABITZ_RCLS:R-0603
- added R19, R21, R22, R41, R6, R7: 21K, HEXABITZ_RCLS:R-0603
- added R23: 2.4M, HEXABITZ_RCLS:R-0603
- added R24, R27, R29, R57: 12K, HEXABITZ_RCLS:R-0603
- added R25: 100K, HEXABITZ_RCLS:R-0603
- added R26, R28, R56: 1K, HEXABITZ_RCLS:R-0603
- added R42, R44, R9: 10.5K, HEXABITZ_RCLS:R-0603
- added R46, R48, R49: 2.2K, HEXABITZ_RCLS:R-0603
- added R47: 18K, HEXABITZ_RCLS:R-0603
- added R50, R51: DNP, HEXABITZ_RCLS:R-0603
- added R52: 0R, HEXABITZ_RCLS:R-0603
- added R53: 270R, HEXABITZ_RCLS:R-0603
- added R54: 180K, HEXABITZ_RCLS:R-0603
- added R55: 10K, HEXABITZ_RCLS:R-0603
- added U2: STSPIN32F0A, HEXABITZ_ICs:STSPIN32F0A
- added U3: AM26LV32EIRGYRTEXAS_INSTRUMENTS_AM26LV32EIRGYR_0_0, HEXABITZ_ICs:AM26LV32EIRGYRTEXAS_INSTRUMENTS_AM26LV32EIRGYR_0_0
- added U4: NCP730BMTADJTBGON_SEMI_NCP730BMTADJTBG_0_0, HEXABITZ_ICs:NCP730BMTADJTBGON_SEMI_NCP730BMTADJTBG_0_0
Connections:
- removed net VSSA: C2.1, C3.-, C4.1, C5.-, R1.2, U1.VSS/VSSA
- new net +5V: C25.2, C26.2, C32.1, C33.1, J3.2, J4.2, R23.1, U4.OUT
- new net ENC_A: J3.4, U3.1A
- new net ENC_B: J3.6, U3.4A
- new net ENC_I: J3.8, U3.3A
- new net ENC_NA: J3.3, U3.1B
- new net ENC_NB: J3.5, U3.4B
- new net ENC_NI: J3.7, U3.3B
- new net G0_USART1_RX: U1.PA10, U2.PB6
- new net G0_USART1_TX: U1.PA9, U2.PA15
- new net GND1: C11.2, C12.2, C13.2, C14.1, C15.2, C16.2, C17.1, C18.1, C19.1, C2.1, C20.2, C21.2, C22.2, C23.1, C24.1, C25.1, C27.1, C28.1, C29.1, C3.-, C30.-, C31.-, C32.2, C33.2, C4.1, C45.1, C46.1, C5.-, D10.C, D8.ANODE, GND.P$1, J2.2, J3.1, J4.4, J4.6, R1.2, R10.1, R12.2, R14.1, R17.1, R18.1, R21.2, R25.2, R41.2, R43.1, R45.1, R55.1, R6.2, U1.VSS/VSSA, U2.EPAD, U2.GND, U2.TESTMODE, U3.!G!, U3.EP, U3.GND, U4.EP, U4.GND
- new net H1: J4.1, R56.1, R57.2
- new net H2: J4.3, R26.1, R27.2
- new net H3: J4.5, R28.1, R29.2
- new net HSU: D3.C, R5.2, U2.HSU
- new net HSV: D5.C, R13.2, U2.HSV
- new net HSW: D7.C, R16.2, U2.HSW
- new net ISNSU: Q1G$1.S1, R10.2, R40.1, R46.2
- new net ISNSV: Q2G$1.S1, R14.2, R20.1, R48.2
- new net ISNSW: Q3G$1.S1, R17.2, R49.2, R8.1
- new net LSU: D2.C, R4.2, U2.LSU
- new net LSV: D4.C, R11.2, U2.LSV
- new net LSW: D6.C, R15.2, U2.LSW
- new net N$10: D4.A, Q2G$1.G1, R11.1
- new net N$11: C26.1, R12.1, R23.2, U4.ADJ
- new net N$13: D3.A, Q1G$2.G2, R5.1
- new net N$14: C27.2, R24.1, U2.NRST
- new net N$15: C13.1, U2.VREG12
- new net N$16: D5.A, Q2G$2.G2, R13.1
- new net N$17: BOOT0.P$1, R25.1, U2.BOOT0
- new net N$18: U3.2A
- new net N$26: D6.A, Q3G$1.G1, R15.1
- new net N$27: D7.A, Q3G$2.G2, R16.1
- new net N$29: R18.2, R9.1, U2.OP1N
- new net N$30: R44.1, R45.2, U2.OP3N
- new net N$31: C19.2, R46.1, R47.2, R48.1, R49.1, U2.OC_COMP
- new net N$32: D10.A, R53.1
- new net N$33: D8.CATHODE, FB2.1, R50.2, U2.SW
- new net N$34: C20.1, FB2.2, R52.1
- new net N$5: R42.1, R43.2, U2.OP2N
- new net N$6: C8.2, U2.VBOOTU
- new net N$7: C9.2, U2.VBOOTV
- new net N$8: C10.2, U2.VBOOTW
- new net N$9: D2.A, Q1G$1.G1, R4.1
- new net OP1P: C14.2, R6.1, R7.2, R8.2, U2.OP1P
- new net OP2P: C18.2, R22.2, R40.2, R41.1, U2.OP2P
- new net OP3P: C17.2, R19.2, R20.2, R21.1, U2.OP3P
- new net OUTU: C8.1, J1.1, Q1G$1.D1, Q1G$2.S2, U2.OUTU
- new net OUTV: C9.1, J1.2, Q2G$1.D1, Q2G$2.S2, U2.OUTV
- new net OUTW: C10.1, J1.3, Q3G$1.D1, Q3G$2.S2, U2.OUTW
- new net PA0: C46.2, R56.2, U2.PA0
- new net PA1: C28.2, R26.2, U2.PA1
- new net PA2: C29.2, R28.2, U2.PA2
- new net PA3: R42.2, U2.OP2O, U2.PA3
- new net PA4: R44.2, U2.OP3O, U2.PA4
- new net PA5: R9.2, U2.OP1O, U2.PA5
- new net PA6: U2.PA6, U3.1Y
- new net PA7: U2.PA7, U3.4Y
- new net PB1: C45.2, R54.2, R55.2, U2.PB1
- new net PF0: R53.2, U2.PF0
- new net PF1: U2.PF1, U3.3Y
- new net SWDCLK: SWDCLK.P$1, U2.PA14_SWD_CLK
- new net SWDIO: SWDIO.P$1, U2.PA13_SWD_IO
- new net VDD_L: C21.1, C22.1, C23.2, R19.1, R22.1, R24.2, R27.1, R29.1, R47.1, R51.2, R52.2, R57.1, R7.1, U2.VDD, U2.VDDA, U3.2B, U3.G, U3.VCC
- new net VM: C11.1, C12.1, C15.1, C16.1, C24.2, C30.+, C31.+, J2.1, Q1G$2.D2, Q2G$2.D2, Q3G$2.D2, R50.1, R54.1, U2.VM, U4.EN, U4.IN
- net VDD: now also R51.1
Other:
- note added: "3"
- note added: "5V LDO"
- note added: "Driver Outupt"
- note added: "Encoder Input"
- note added: "Hall-effect Sensor"
- note added: "VM = 12-38V"
