File: H19R00/Design/H19R00.sch (EAGLE design)
At the start: 112 parts, among them J1 691213710003, J2 691213710002, J3 20021121-00008T4LFU, J4 20021121-00006C1LF, U1 STM32G0B1CEU6N, U2 STSPIN32F0A, U3 AM26LV32EIRGYRTEXAS_INSTRUMEN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, U4 NCP730BMTADJTBGON_SEMI_NCP730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, X1 8MHZ

Commit message: -Add some notes to the schematic -fix the BOM - Add NRST,TX1 and RX1  test points -Fix some issues at the silkscreen layer
Parts:
- added NRST, RX1, TX1: PAD4, HEXABITZ_CONNECTION_PARTS:PAD4
Connections:
- net G0_USART1_RX: now also RX1.P$1
- net G0_USART1_TX: now also TX1.P$1
- net GND: no longer U1.PA0, U1.PA1
- net N$14: now also NRST.P$1
Other:
- note added: "36 V/6A Sensored BLDC"
- note added: "Do not supply any other circuits from this connector except the Hall-effect Sensor. (maximum drawn current should not exceed 150 mA)"
- note added: "Do not supply any other circuits from this connector except the encoder. (maximum drawn current should not exceed 150 mA)"
- note added: "If you want to use this module as stnadalone without providing external 3V3 you have to remove the jumber resistor and place the 2 DNP resistors. Attention : make sure (in this situatoin) you didn't connect any other modules to this module (the dranw current form the Vdd pads doesn't exceed 100mA)."
- note added: "Muhammad Awais"
- note removed: "36 V/6 Apeak Brushless DC"
- moved on the sheet: C27

Commit message: -Fix the BOM and some parts attributes
Parts:
- C10, C8, C9: MFN KYOCERA AVX -> TDK Corporation; MPN 06031C471K4T2A -> C1608X5R1H474K080AB; OCTOPART_URL https://octopart.com/search?q=06031C471K4T2A&currency=USD&s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 -> https://octopart.com/search?q=C1608X5R1H474K080AB&currency=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; VOLTAGE_RATING 100V -> 50V
Changed lines of the file:
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@@
 <drawing>
 <settings>
-<setting alwaysvectorfont="no"/>
+<setting alwaysvectorfont="yes"/>
 <setting verticaltext="up"/>
 </settings>
-<grid distance="12.5" unitdist="mil" unit="mil" style="lines" multiple="1" display="no" altdistance="0.01" altunitdist="inch" altunit="inch"/>
+<grid distance="0.1" unitdist="inch" unit="inch" style="lines" multiple="1" display="no" altdistance="0.01" altunitdist="inch" altunit="inch"/>
 <layers>
 <layer number="1" name="Top" color="4" fill="1" visible="no" active="no"/>
@@
 <part name="C8" library="HEXABITZ_RCLS" library_urn="urn:adsk.eagle:library:20064561" deviceset="C-0603" device="" package3d_urn="urn:adsk.eagle:package:19666468/3" value="470nF">
 <attribute name="CAPACITANCE" value="470nF"/>
-<attribute name="MFN" value="KYOCERA AVX"/>
-<attribute name="MPN" value="06031C471K4T2A"/>
-<attribute name="OCTOPART_URL" value="https://octopart.com/search?q=06031C471K4T2A&amp;currency=USD&amp;specs=0"/>
-<attribute name="TOLERANCE" value="10%"/>
-<attribute name="VOLTAGE_RATING" value="100V"/>
+<attribute name="MFN" value="TDK Corporation"/>
+<attribute name="MPN" value="C1608X5R1H474K080AB"/>
+<attribute name="OCTOPART_URL" value="https://octopart.com/search?q=C1608X5R1H474K080AB&amp;currency=USD&amp;specs=0"/>
+<attribute name="TOLERANCE" value="10%"/>
+<attribute name="VOLTAGE_RATING" value="50V"/>
 </part>
 <part name="C9" library="HEXABITZ_RCLS" library_urn="urn:adsk.eagle:library:20064561" deviceset="C-0603" device="" package3d_urn="urn:adsk.eagle:package:19666468/3" value="470nF">
 <attribute name="CAPACITANCE" value="470nF"/>
-<attribute name="MFN" value="KYOCERA AVX"/>
-<attribute name="MPN" value="06031C471K4T2A"/>
-<attribute name="OCTOPART_URL" value="https://octopart.com/search?q=06031C471K4T2A&amp;currency=USD&amp;specs=0"/>
-<attribute name="TOLERANCE" value="10%"/>
-<attribute name="VOLTAGE_RATING" value="100V"/>
+<attribute name="MFN" value="TDK Corporation"/>
+<attribute name="MPN" value="C1608X5R1H474K080AB"/>
+<attribute name="OCTOPART_URL" value="https://octopart.com/search?q=C1608X5R1H474K080AB&amp;currency=USD&amp;specs=0"/>
+<attribute name="TOLERANCE" value="10%"/>
+<attribute name="VOLTAGE_RATING" value="50V"/>
 </part>
 <part name="C10" library="HEXABITZ_RCLS" library_urn="urn:adsk.eagle:library:20064561" deviceset="C-0603" device="" package3d_urn="urn:adsk.eagle:package:19666468/3" value="470nF">
 <attribute name="CAPACITANCE" value="470nF"/>
-<attribute name="MFN" value="KYOCERA AVX"/>
-<attribute name="MPN" value="06031C471K4T2A"/>
-<attribute name="OCTOPART_URL" value="https://octopart.com/search?q=06031C471K4T2A&amp;currency=USD&amp;specs=0"/>
-<attribute name="TOLERANCE" value="10%"/>
-<attribute name="VOLTAGE_RATING" value="100V"/>
+<attribute name="MFN" value="TDK Corporation"/>
+<attribute name="MPN" value="C1608X5R1H474K080AB"/>
+<attribute name="OCTOPART_URL" value="https://octopart.com/search?q=C1608X5R1H474K080AB&amp;currency=USD&amp;specs=0"/>
+<attribute name="TOLERANCE" value="10%"/>
+<attribute name="VOLTAGE_RATING" value="50V"/>
 </part>
 <part name="D2" library="HEXABITZ_RCLS" library_urn="urn:adsk.eagle:library:20064561" deviceset="BAT30KFILM" device="" package3d_urn="urn:adsk.eagle:package:41622969/2"/>
