File: H19R00/Design/H19R00.brd (EAGLE design)
At the start: 60 x 60.6 mm, 115 parts, among them J1 691213710003, J2 691213710002, J3 20021121-00008T4LFU, J4 20021121-00006C1LF, U1 STM32G0B1CEU6N, U2 STSPIN32F0A, U3 AM26LV32EIRGYRTEXAS_INSTRUMEN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, U4 NCP730BMTADJTBGON_SEMI_NCP730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, X1 8MHZ

Commit message: All the edits that is related to 10A handling is done : -Improve the layout design so the pcb can handle continous current up to 10A -Naming the smd pin headers and thier pins on the silk screen layer -Change the high voltage supply coupling smd capacitors to dip ones with bigger capacity - Edit the resistores values of the current sensing and comparator circuits to be compitable with the 10A and add the equtions as notes in the schematic
Parts:
- C30, C31: device HEXABITZ_RCLS:PANASONIC_D -> HEXABITZ_RCLS:CAPPRD350W60D825H1300
- R10, R14, R17: value 0.100R -> 0.050R
- R19, R21, R22, R41, R6, R7: value 21K -> 14.3K
- R42, R44, R9: value 10.5K -> 7.15K
- R46, R48, R49: value 2.2K -> 0.51K
- R47: value 18K -> 200K
- moved D10 5.23 mm to (25.1, 16.4), turned to 90 degrees
- moved R53 4.34 mm to (23.0, 17.3)
- moved C33 4.30 mm to (-12.5, 25.7), turned to 90 degrees
- moved C30 2.84 mm to (-19.7, 0.16), turned to 180 degrees
- moved C31 1.87 mm to (-22.7, 8.71), turned to 180 degrees
- moved C32 1.09 mm to (10.1, 22.6), turned to 180 degrees
- moved C23 0.71 mm to (10.1, 24.2)
Connections:
- net GND1: now also C30.2, C31.2; no longer C30.-, C31.-
- net VM: now also C30.1, C31.1; no longer C30.+, C31.+
Routing:
- net GND1: track 107.0 -> 102.7 mm, vias 80 -> 79
- net PF0: track 33.3 -> 35.0 mm
- net ENC_NB: track 16.2 -> 17.1 mm
- net ENC_B: track 14.3 -> 15.0 mm
- net VDD_L: track 121.8 -> 122.5 mm
- added copper zone on layer 15, net OUTU
- added copper zone on layer 15, net OUTV
- added copper zone on layer 15, net OUTW
- added copper zone on layer 16, net VM
- removed copper zone on layer 2, net VM
Other:
- board text added: "+5V"
- board text added: "10A MAX"
- board text added: "A"
- board text added: "ENC_IN"
- board text added: "H1"
- board text added: "H2"
- board text added: "H3"
- board text added: "Hall_Sen"
- board text added: "I"
- board text added: "NA"
- board text added: "NB"
- board text added: "NI"
- board text removed: "6A MAX"
